Commit message: avance2

File: description/properties.xacro (robot description, xacro)
@@ -14,3 +14,6 @@
         <color rgba= "0 0 0 1"/>
     </material>
+        <material name="red">
+        <color rgba= "1 0 0 1"/>
+    </material>
 </robot>

File: description/robot.urdf.xacro (robot description, xacro)
@@ -4,4 +4,8 @@
     <xacro:include filename="properties.xacro"/>
     <xacro:include filename="robot_core.xacro"/>
-    <xacro:include filename="inertial_core_xacro"/>
+    <xacro:include filename="inertial_macros.xacro"/>
+    <xacro:include filename="gazebo_control.xacro"/>
+    <xacro:include filename="lidar.xacro"/>
+    <xacro:include filename="imu.xacro"/>
+    <xacro:include filename="camera.xacro"/>
 </robot>

File: description/robot_core.xacro (robot description, xacro)
@@ -30,4 +30,7 @@
         </xacro:inertial_box>
     </link>
+    <gazebo reference="chassis">
+        <material>Gazebo/White</material>
+    </gazebo>
     <!-- left wheel joint -->
     <joint name="left_wheel_joint" type="continuous">
@@ -54,4 +57,7 @@
         </xacro:inertial_cylinder>
     </link>
+    <gazebo reference="left_wheel">
+        <material>Gazebo/Blue</material>
+    </gazebo>
     <!-- right wheel joint -->
     <joint name="right_wheel_joint" type="continuous">
@@ -78,4 +84,7 @@
         </xacro:inertial_cylinder>
     </link>
+    <gazebo reference="right_wheel">
+        <material>Gazebo/Blue</material>
+    </gazebo>
     <!-- caster wheel joint -->
     <joint name="caster_wheel_joint" type="fixed">
@@ -101,3 +110,8 @@
         </xacro:inertial_sphere>
     </link>
+    <gazebo reference="caster_wheel">
+        <material>Gazebo/Black</material>
+        <mu1 value = "0.001" />
+        <mu2 value = "0.001" />
+    </gazebo>
 </robot>
